Commit message: added two gimbal camera versions with two different mass properties. deleted the old one.

File: rotors_description/urdf/multirotor_base.xacro (robot description, xacro)
@@ -91,5 +91,5 @@
       <visual>
         <geometry>
-          <!-- <cylinder length="0.005" radius="${radius_rotor}"/> --> <!-- [m] -->
+                  <!-- <cylinder length="0.005" radius="${radius_rotor}"/> --> <!-- [m] -->
           <xacro:if value="${use_own_mesh}">
             <mesh filename="${mesh}"
