Commit message: added dji visuals to the pelican robot model (urdf) with stationary propellers

File: rotors_description/urdf/pelican.xacro (robot description, xacro)
@@ -22,8 +22,8 @@
   <xacro:property name="rotor_velocity_slowdown_sim" value="10" />
   <xacro:property name="use_mesh_file" value="true" />
-  <xacro:property name="mesh_file" value="package://rotors_description/meshes/pelican.dae" />
+  <xacro:property name="mesh_file" value="package://rotors_description/meshes/dji_matrice_210_v3_chassis.dae" />
   <xacro:property name="mass" value="1.0" /> <!-- [kg] -->
   <xacro:property name="body_width" value="0.1" /> <!-- [m] -->
-  <xacro:property name="body_height" value="0.2" /> <!-- [m] -->
+  <xacro:property name="body_height" value="0.54" /> <!-- [m] -->
   <xacro:property name="mass_rotor" value="0.01" /> <!-- [kg] -->
   <xacro:property name="arm_length" value="0.21" /> <!-- [m] -->
@@ -74,5 +74,5 @@
     rolling_moment_coefficient="${rolling_moment_coefficient}"
     color="Red"
-    use_own_mesh="false"
+    use_own_mesh="true"
     mesh="">
     <origin xyz="${arm_length} 0 ${rotor_offset_top}" rpy="0 0 0" />
@@ -95,5 +95,5 @@
     rolling_moment_coefficient="${rolling_moment_coefficient}"
     color="Blue"
-    use_own_mesh="false"
+    use_own_mesh="true"
     mesh="">
     <origin xyz="0 ${arm_length} ${rotor_offset_top}" rpy="0 0 0" />
@@ -116,5 +116,5 @@
     rolling_moment_coefficient="${rolling_moment_coefficient}"
     color="Blue"
-    use_own_mesh="false"
+    use_own_mesh="true"
     mesh="">
     <origin xyz="-${arm_length} 0 ${rotor_offset_top}" rpy="0 0 0" />
@@ -137,5 +137,5 @@
     rolling_moment_coefficient="${rolling_moment_coefficient}"
     color="Blue"
-    use_own_mesh="false"
+    use_own_mesh="true"
     mesh="">
     <origin xyz="0 -${arm_length} ${rotor_offset_top}" rpy="0 0 0" />
